File: diag.kicad_pcb (KiCad board)
At the start: 2 copper layers, 101.6 x 99.3 mm, 67 parts, among them CN1 DRAGON-EDGE-CONN, CN2 JTAG-CONN2X3, IC1 29F040, IC2 32KSRAM-DIL600, IC3 XC9572XL-TQ100

Commit message: convert files to kicad, change to 4 layers and supplement decoupling
Parts:
- added C10: 0.01µf, Capacitor_SMD:C_0805_2012Metric, F.Cu at (137.4, 99.9)
- added C8: 0.01µf, Capacitor_SMD:C_0805_2012Metric, F.Cu at (147.1, 74.5)
- added C9: 0.01µf, Capacitor_SMD:C_0805_2012Metric, F.Cu at (155.5, 87.9)
- C4, C5, C6, C7: footprint diag:C025-025X050 -> Capacitor_SMD:C_0805_2012Metric
- DS1, DS2, DS3: value (none) -> DIP04S
- IC3: value XC9572XL-TQ100 -> XC95144XL-TQ100
- JP5: value (none) -> PINHD-1X4
- JP6, JP7, JP8: value (none) -> PINHD-1X2
- JP9: value (none) -> PINHD-1X3
- P19, P2, P24, P29, P7, P80, P85: value (none) -> PINHD-1X1
- REG1B0: value LT1963EST-3.3 -> LT1963EST; footprint diag:SOT223 -> PCM_Package_TO_SOT_SMD_AKL:SOT-223-3_TabPin2
- S1, S2, S3, S4, S5: value (none) -> 10-XX
- moved C7 5.36 mm to (130.6, 87.2)
- moved C4 0.87 mm to (133.4, 96.7), turned to -90 degrees
- moved RN3 0.45 mm to (144.5, 150.7)
- moved C6 0.29 mm to (153.2, 79.6), turned to 0 degrees
- turned C5 to 0 degrees
- turned REG1B0 to 180 degrees
Connections:
- net +12V renamed /diag_1/+12V
- net -12V renamed /diag_1/-12V
- net AS renamed /diag_2/AS
- net BL+ renamed /diag_1/BL+
- net CONT renamed /diag_1/CONT
- net P19 renamed /diag_2/P19
- net P2 renamed /diag_2/P2
- net P24 renamed /diag_2/P24
- net P29 renamed /diag_2/P29
- net P34 renamed /diag_2/P34
- net P43 renamed /diag_2/P43
- net P46 renamed /diag_2/P46
- net P7 renamed /diag_2/P7
- net P80 renamed /diag_2/P80
- net P85 renamed /diag_2/P85
- net R/~{W} renamed R/~{W}
- net ROMA14 renamed /diag_1/ROMA14
- net ROMA15 renamed /diag_1/ROMA15
- net ROMA16 renamed /diag_1/ROMA16
- net ROMA17 renamed /diag_1/ROMA17
- net S1 renamed /diag_2/S1
- net S2 renamed /diag_2/S2
- net S3 renamed /diag_2/S3
- net S4 renamed /diag_2/S4
- net SP0 renamed /diag_2/SP0
- net SP1 renamed /diag_2/SP1
- net SP2 renamed /diag_2/SP2
- net SP3 renamed /diag_2/SP3
- net TCK renamed /diag_2/TCK
- net TDI renamed /diag_2/TDI
- net TDO renamed /diag_2/TDO
- net TMS renamed /diag_2/TMS
- net ~{DIS_REMAP} renamed /diag_2/~{DIS_REMAP}
- net ~{RESET} renamed /diag_1/~{RESET}
- net ~{ROMWE} renamed /diag_1/~{ROMWE}
- CN1 pad P35: (no net) -> unconnected-(CN1-SND-PadP35)
- S1 pad 1: (no net) -> unconnected-(S1-S-Pad1)
- S1 pad 4: (no net) -> unconnected-(S1-P1-Pad4)
- S2 pad 1: (no net) -> unconnected-(S2-S-Pad1)
- S2 pad 4: (no net) -> unconnected-(S2-P1-Pad4)
- S3 pad 1: (no net) -> unconnected-(S3-S-Pad1)
- S3 pad 4: (no net) -> unconnected-(S3-P1-Pad4)
- S4 pad 1: (no net) -> unconnected-(S4-S-Pad1)
- S4 pad 4: (no net) -> unconnected-(S4-P1-Pad4)
Routing:
- net GND: track 546.3 -> 50.2 mm, vias 3 -> 25
- net VCC33: track 321.0 -> 42.2 mm, vias 1 -> 7
- net /diag_2/P85: track 40.3 -> 19.6 mm
- net /diag_2/P19: track 54.6 -> 39.6 mm
- net /diag_1/BL+: track 37.4 -> 25.6 mm
- net R/~{W}: track 125.4 -> 119.5 mm
- net /diag_2/TDO: track 35.7 -> 30.4 mm
- net D3: track 178.7 -> 173.8 mm
- net ~{DSD}: track 86.2 -> 81.6 mm
- net ~{P2}: track 86.8 -> 82.4 mm
- net /diag_2/S4: track 90.8 -> 94.9 mm
- net /diag_2/S3: track 78.5 -> 82.3 mm
- net D7: track 166.7 -> 163.3 mm
- net /diag_2/S2: track 75.5 -> 78.8 mm
- net /diag_2/S1: track 74.4 -> 77.7 mm
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- added copper zone on In1.Cu, net GND
- added copper zone on In2.Cu, net VCC33
Other:
- board size 101.6 x 99.3 mm -> 101.7 x 99.3 mm
- copper layers 2 -> 4

Commit message: convert more passives to smd
Parts:
- removed JP1, JP2, JP3, JP4: STAND-OFF, diag:STAND-OFF
- removed REG1A0: LEXXCZ, diag:TO92-
- D1: value 1N4148DO35-7 -> 1N4148WS; footprint diag:DO35-7 -> Diode_SMD:D_SOD-323
- R10, R11, R12, R13, R14, R2, R4, R5, R6, R7, R8, R9: footprint diag:0207_10 -> PCM_Resistor_SMD_AKL:R_0805_2012Metric
- R3: footprint diag:0204_7 -> PCM_Resistor_SMD_AKL:R_0805_2012Metric
- moved R14 13.2 mm to (141.0, 145.1), turned to 180 degrees
- moved R13 7.44 mm to (176.6, 69.6)
- moved R11 5.12 mm to (185.9, 134.2), turned to 180 degrees
- moved R5 4.85 mm to (188.1, 74.5)
- moved R7 4.43 mm to (188.1, 78.0)
- moved R8 4.19 mm to (188.2, 66.2)
- moved R9 4.19 mm to (188.2, 59.3)
- moved R6 4.19 mm to (188.2, 62.8)
- moved R10 4.18 mm to (188.1, 81.5)
- moved R4 4.15 mm to (188.1, 71.1)
- moved R12 4.13 mm to (126.2, 62.5)
- moved R3 2.99 mm to (117.8, 82.7)
- moved D1 1.50 mm to (114.7, 87.3)
- moved JP6 0.67 mm to (175.7, 61.2)
- moved JP7 0.67 mm to (175.7, 66.3)
Routing:
- net /diag_1/+12V: track 108.5 -> 122.8 mm, vias 0 -> 1
- net RSTLED: track 54.1 -> 62.3 mm
- net HLTLED: track 36.5 -> 43.9 mm, vias 0 -> 2
- net ELED: track 37.7 -> 43.7 mm, vias 0 -> 2
- net VCC: track 317.6 -> 311.7 mm, vias 2 -> 5
- net /diag_1/-12V: track 118.9 -> 113.3 mm, vias 0 -> 1
- net QLED: track 38.6 -> 44.0 mm, vias 0 -> 2
- net /diag_2/S1: track 77.7 -> 72.8 mm
- net /diag_2/S2: track 78.8 -> 74.1 mm
- net Net-(JP9-Pad3): track 8.25 -> 3.73 mm
- net /diag_2/S3: track 82.3 -> 77.8 mm
- net /diag_2/S4: track 94.9 -> 90.6 mm
- net /diag_1/BL+: track 25.6 -> 29.7 mm, vias 0 -> 1
- net R/~{W}: track 119.5 -> 115.4 mm
- net /diag_1/~{RESET}: track 4.71 -> 8.64 mm
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Other:
- board text added: "-5/12V"
- board text removed: "-12V"

Commit message: tidy-up
Parts:
- added JP1: STAND-OFF, diag:STAND-OFF, F.Cu at (108.1, 58.7)
- added JP2: STAND-OFF, diag:STAND-OFF, F.Cu at (202.7, 151.4)
- added JP3: STAND-OFF, diag:STAND-OFF, F.Cu at (108.1, 151.4)
- added JP4: STAND-OFF, diag:STAND-OFF, F.Cu at (202.7, 58.7)
- C1, C2: footprint diag:C025-025X050 -> PCM_Capacitor_SMD_AKL:C_0805_2012Metric
- moved C1 6.08 mm to (163.4, 133.2), turned to 90 degrees
- moved C2 2.32 mm to (158.2, 117.7), turned to 90 degrees
- moved R13 0.25 mm to (176.6, 69.8)
Routing:
- net A14: track 102.8 -> 108.9 mm
- net VCC: track 311.7 -> 315.9 mm, vias 5 -> 7
- net GND: track 53.3 -> 56.3 mm, vias 28 -> 30
- net ~{ROMCS}: track 74.9 -> 77.8 mm
- net A15: track 138.0 -> 139.5 mm
Other:
- outline, holes or cut-outs redrawn
